File: hardware/CutDown2/CutDown2_V1/CutDown2_V1.0.sch (EAGLE design)
At the start: 50 parts, among them Q1 2N3906, Q3 2N3906, Q4 2N3906, T1 2N3904, T2 2N3904, T4 2N3904, U1 ADCMP354OC, U2 ADCMP354OC, U3 LM60

Commit message: Updates
Parts:
- removed D2: BZX85, diode:BZX85
- removed D3, D5, D6: 1N5817-B, diode:1N5817-B
- removed JP1: (no value), adafruit:PINHD-1X6
- removed LED3, LED4: (no value), eagle-ltspice:LED_ELD260
- removed PAD1, PAD2, PAD3: (no value), wirepad:2,15/1,0
- removed R10: 2k, rcl:R-US_0207/7
- removed R12, R15: 3.9k, rcl:R-US_0207/7
- removed R13, R21: 39k, rcl:R-US_0207/7
- removed R14: 12k, rcl:R-US_0207/7
- removed R16, R6: 1k, rcl:R-US_0207/7
- removed R18: 300, rcl:R-US_0207/7
- removed R20: 51k, rcl:R-US_0207/7
- removed R9: 22k, rcl:R-US_0207/7
- removed S2: SWS002, smd-special:SWS002
- removed T1, T2, T4: 2N3904, transistor:2N3904
- removed U$1, U$2: BH1000G, mymechanical:BH1000G
- removed U$3: 1.5F, mypassives:C1000X850
- removed U$4: ARDUINOMINI, adafruit:ARDUINOMINI
- removed U1, U2: ADCMP354OC, mydevices:ADCMP354OC
- added A1: XBEE, adafruit:XBEE
- added A2: ARDUINOMINI3.3V, fhdevices:ARDUINOMINI3.3V
- added B1: 9V_BATT, fhmechanical:9V_BATT
- added D1: 1N5817-B, diode:1N5817-B
- added JP2: (no value), SparkFun-Connectors:M03POLAR_LOCK
- added M1: RS_BOX_4IN, mymechanical:RS_BOX_4IN
- added M2: 9V_BATT_CLIP, fhmechanical:9V_BATT_CLIP
- added Q2: MMBT3904, SparkFun-DiscreteSemi:TRANSISTOR_NPNSOT23
- added S1: APEM_SPDT_25000NH, fhmechanical:APEM_SPDT_25000NH
- Q1, Q3: value 2N3906 -> MMBT3906; device transistor-pnp:2N3906 -> SparkFun-DiscreteSemi:TRANSISTOR_PNPMMBT4403
- Q4: value 2N3906 -> MMBT3904; device transistor-pnp:2N3906 -> SparkFun-DiscreteSemi:TRANSISTOR_NPNSOT23
- R1, R11, R17, R19, R22, R23, R5, R7, R8: device rcl:R-US_0207/7 -> resistor:R-US_R0805
- R2: value 51k -> 82k; device rcl:R-US_0207/7 -> resistor:R-US_R0805
- R3: value 100k -> 1k; device rcl:R-US_0207/7 -> resistor:R-US_R0805
- R4: value 3.9k -> 10k; device rcl:R-US_0207/7 -> resistor:R-US_R0805
- U3: value LM60 -> LM60_SMD; device mydevices:LM60 -> mydevices:LM60_SMD
Connections:
- removed net N$12: U$1.P2, U$2.P1
- removed net N$14: D6.C, Q3.E
- removed net N$15: D2.C, R10.1, U1.VCC, U2.VCC
- removed net N$16: R13.1, R14.2, U2.IN
- removed net N$17: LED3.C, R3.1, U2.OUT
- removed net N$18: LED3.A, R12.1
- removed net N$19: LED4.A, R15.1
- removed net N$20: LED4.C, R16.1, T2.C
- removed net N$23: Q4.B, R16.2
- removed net N$25: U$4.A5, U3.VO
- removed net N$27: Q4.C, R18.2
- removed net N$28: D5.C, Q4.E
- removed net N$29: JP1.1, U$4.HDTR
- removed net N$30: U$4.VCC0, U3.+VS
- removed net N$32: JP1.2, U$4.HTXO
- removed net N$34: R21.1, R22.2, R9.2
- removed net N$36: D5.A, D6.A, R10.2, R12.2, R15.2, R4.2, R5.2, S2.1
- removed net N$38: D4.A, R2.2, S2.4, U$1.P1
- removed net N$39: JP1.3, U$4.HRXI
- removed net N$40: JP1.6, U$4.HGND
- removed net VBSNS: R13.2, R20.1, U$4.A3
- new net 9V: B1.V+, D4.A, R2.2
- new net VCC: A1.VCC, A2.V3.3, U3.+VS
- net GND: now also A1.GND, A2.GND, A2.GND1, B1.V-, JP2.3, LED1.C, LED2.C, Q2.E, Q4.E; no longer D2.A, PAD2.P, R14.1, T1.E, T2.E, T4.E, U$2.P2, U$3.2, U$4.GND0, U$4.GND1, U1.GND, U2.GND
- net N$1: now also Q3.B, R3.1; no longer U1.IN
- net N$10: now also A1.DIN, A2.TXO; no longer D3.A, R18.1, R20.2, U$3.1
- net N$11: now also S1.P; no longer D3.C, S2.3
- net N$13: now also Q2.B; no longer T1.B
- net N$2: now also D1.A; no longer R8.2
- net N$21: now also Q4.C; no longer T4.C
- net N$24: now also JP2.1; no longer PAD3.P
- net N$26: now also A2.D10; no longer U$4.D10
- net N$3: now also A2.D8, R5.2; no longer LED1.C, U1.OUT
- net N$31: now also Q4.B; no longer T4.B
- net N$41: now also JP2.2; no longer PAD1.P
- net N$42: now also A2.RAW, Q3.E, R4.2, S1.2; no longer S2.2, U$4.RAW
- net N$5: now also A2.A0, R22.2, R23.1; no longer LED2.A, R4.1
- net N$6: now also D1.C, R8.2; no longer LED2.C, R6.1, T1.C
- net N$7: now also LED2.A, Q2.C, R3.2, R4.1; no longer Q3.B, R6.2
- net N$8: now also A1.DOUT, A2.RXI; no longer R9.1, U$4.D9
- net N$9: now also A2.A3, U3.VO; no longer R3.2, T2.B
- net VBATTSNS: now also A2.A2; no longer U$4.A4
- net VCSNS: now also A1.DTR/DI8, A2.D7; no longer R21.2, R23.1, U$4.A2
Other:
- note added: "To-Do: Lengthen wires so lid opens further and battery is easy to change. Change charging resistor back to 100 ohms."
- moved on the sheet: D4, LED1, LED2, R3, R4, R5, R7, R8, U3
