File: hardware/CutDownTimer/ChargerTimer_V5.brd (EAGLE design)
At the start: 92.5 x 41.8 mm, 50 parts, among them Q1 2N3906, Q3 2N3906, Q4 2N3906, T1 2N3904, T2 2N3904, T4 2N3904, U1 ADCMP354OC, U2 ADCMP354OC, U3 LM60

Commit message: Updates
Parts:
- removed D2: BZX85, diode:DO41Z10
- removed D3, D5, D6: 1N5817-B, diode:DO41-7.6
- removed LED3, LED4: (no value), eagle-ltspice:LED_LD260
- removed Q4: 2N3906, transistor-pnp:TO92
- removed R10: 2k, rcl:0207/7
- removed R12, R15: 3.9k, rcl:0207/7
- removed R13, R21: 39k, rcl:0207/7
- removed R14: 12k, rcl:0207/7
- removed R16: 1k, rcl:0207/7
- removed R18: 300, rcl:0207/7
- removed R20: 51k, rcl:0207/7
- removed R3: 100k, rcl:0207/7
- removed R9: 22k, rcl:0207/7
- removed T2: 2N3904, transistor:TO92
- removed U$2: BH1000G, mymechanical:BH1000G
- removed U$3: 1.5F, mypassives:SUPERCAP1.0/0.85H
- removed U1, U2: ADCMP354OC, mydevices:ADCMP35X
- R1: value 39k -> 27k
- R2: value 51k -> 75k
- R22: value 27k -> 68k
- R23: value 51k -> 33k
Connections:
- removed net N$1: U1.P1
- removed net N$12: U$1.NEG$2, U$2.POS$1
- removed net N$14: D6.C, Q3.3
- removed net N$15: D2.C, R10.1, U1.P4, U2.P4
- removed net N$16: R13.1, R14.2, U2.P1
- removed net N$17: LED3.K, R3.1, U2.P3
- removed net N$18: LED3.A, R12.1
- removed net N$19: LED4.A, R15.1
- removed net N$20: LED4.K, R16.1, T2.1
- removed net N$23: Q4.2, R16.2
- removed net N$26: R11.2, U$4.P$30
- removed net N$27: Q4.1, R18.2
- removed net N$28: D5.C, Q4.3
- removed net N$34: R21.1, R22.2, R9.2
- removed net N$36: D5.A, D6.A, R10.2, R12.2, R15.2, R4.2, R5.2, S2.1
- removed net N$42: Q1.3, R19.2, S2.2, U$4.P$19
- removed net VBSNS: R13.2, R20.1, U$4.P$23
- new net N$37: R1.1, U$1.NEG$2, U$4.P$20, U$4.P$9, U3.3
- net GND: no longer D2.A, PAD2.1, R1.1, R14.1, R22.1, T2.3, U$2.NEG$2, U$3.P$2, U$4.P$20, U$4.P$9, U1.P2, U2.P2, U3.3
- net N$10: now also R11.1, U$4.P$8; no longer D3.A, R18.1, R20.2, U$3.P$1
- net N$11: now also Q1.3, Q3.3, R19.2, R2.2, R4.2, R5.2, S2.2, U$4.P$19; no longer D3.C, D4.C, S2.3
- net N$3: now also U$4.P$2; no longer U1.P3
- net N$31: now also R11.2; no longer R11.1
- net N$38: no longer R2.2, S2.4
- net N$8: now also D4.C, S2.3; no longer R9.1, U$4.P$1
- net N$9: now also PAD2.1, R22.1; no longer R3.2, T2.2
- net VBATTSNS: now also U$4.P$23; no longer U$4.P$34
- net VCSNS: now also R22.2; no longer R21.2
Routing:
- net GND: track 131.3 -> 0.00 mm
- net N$10: track 63.3 -> 0.00 mm
- net N$36: track 50.9 -> 0.00 mm
- net N$15: track 37.3 -> 0.00 mm
- net N$12: track 22.3 -> 0.00 mm
- net N$17: track 21.6 -> 0.00 mm
- net N$16: track 16.3 -> 0.00 mm
- net N$18: track 10.7 -> 0.00 mm
- net N$26: track 9.82 -> 0.00 mm
- net N$3: track 24.5 -> 16.7 mm
- net N$20: track 7.33 -> 0.00 mm
- net N$9: track 5.04 -> 0.00 mm
- net N$19: track 3.12 -> 0.00 mm
- net N$1: track 1.63 -> 0.00 mm
